Commit message: #556: updated IMU configuration

File: eufs_sensors/urdf/imu.urdf.xacro (robot description, xacro)
@@ -4,4 +4,5 @@
         <joint name="${prefix}_base_joint" type="fixed">
             <axis xyz="1 0 0"/>
+            <origin xyz="0 0 0" rpy="0 0 0"/>
             <xacro:insert_block name="origin"/>
             <parent link="${parent}"/>
@@ -80,5 +81,5 @@
                         <remapping>~/out:=${prefix}</remapping>
                     </ros>
-                    <frame_name>${prefix}_base_link</frame_name>
+                    <frame_name>${prefix}_base_link_ned</frame_name>
                     <initial_orientation_as_reference>false</initial_orientation_as_reference>
                 </plugin>

Commit message: rotated imu to be enu

File: eufs_sensors/urdf/imu.urdf.xacro (robot description, xacro)
@@ -4,5 +4,5 @@
         <joint name="${prefix}_base_joint" type="fixed">
             <axis xyz="1 0 0"/>
-            <origin xyz="0 0 0" rpy="0 0 0"/>
+            <origin xyz="0 0 0" rpy="0 0 -1.57"/>
             <xacro:insert_block name="origin"/>
             <parent link="${parent}"/>
@@ -81,5 +81,5 @@
                         <remapping>~/out:=${prefix}</remapping>
                     </ros>
-                    <frame_name>${prefix}_base_link_ned</frame_name>
+                    <frame_name>${prefix}_base_link</frame_name>
                     <initial_orientation_as_reference>false</initial_orientation_as_reference>
                 </plugin>
