Commit message: Update velodyne settings

File: eufs_racecar/robots/ads-dv/robot.urdf.xacro (robot description, xacro)
@@ -47,5 +47,5 @@
     </xacro:sensor_gps>
     <xacro:VLP-16R parent="base_footprint" name="velodyne" topic="/velodyne_points" hz="10" samples="800" active="$(arg simulate_perception)">
-	<origin xyz="0.59 0.0 0.51" rpy="0 ${10*M_PI/180.0} 0"/>
+	<origin xyz="0.59 0.0 0.30" rpy="0 0 0"/>
     </xacro:VLP-16R>
     <xacro:zed_camera parent="base_footprint" prefix="zed" active="$(arg simulate_perception)">

File: eufs_racecar/robots/eufs/robot.urdf.xacro (robot description, xacro)
@@ -47,5 +47,5 @@
     </xacro:sensor_gps>
     <xacro:VLP-16R parent="base_footprint" name="velodyne" topic="/velodyne_points" hz="10" active="$(arg simulate_perception)">
-        <origin xyz="-0.15 0.0 0.79" rpy="0 ${1*M_PI/180.0} 0"/>
+        <origin xyz="-0.15 0.0 0.30" rpy="0 0 0"/>
     </xacro:VLP-16R>
     <xacro:zed_camera parent="base_footprint" prefix="zed" active="$(arg simulate_perception)">

File: eufs_sensors/urdf/VLP-16R.urdf.xacro (robot description, xacro)
@@ -2,5 +2,5 @@
 <robot xmlns:xacro="http://www.ros.org/wiki/xacro" name="VLP-16">
   <xacro:property name="M_PI" value="3.1415926535897931" />
-  <xacro:macro name="VLP-16R" params="*origin parent:=base_footprint name:=velodyne active topic:=/velodyne_points hz:=10 lasers:=40 samples:=350 min_range:=0.2 max_range:=100.0 noise:=0.008 min_angle:=-2 max_angle:=2">
+  <xacro:macro name="VLP-16R" params="*origin parent:=velodyne name:=velodyne active topic:=/velodyne_points hz:=10 lasers:=16 samples:=350 min_range:=1.5 max_range:=100.0 noise:=0.008 min_angle:=-2 max_angle:=2">
     <joint name="${name}_base_mount_joint" type="fixed">
       <xacro:insert_block name="origin" />

Commit message: added velodyne lidar plugin and coded up reflectivity of cones

File: eufs_racecar/robots/ads-dv/robot.urdf.xacro (robot description, xacro)
@@ -46,7 +46,10 @@
         <origin xyz="0.0 0.0 0.4" rpy="0 0 0"/>
     </xacro:sensor_gps>
-    <xacro:VLP-16R parent="base_footprint" name="velodyne" topic="/velodyne_points" hz="10" samples="800" active="$(arg simulate_perception)">
-	<origin xyz="0.59 0.0 0.30" rpy="0 0 0"/>
-    </xacro:VLP-16R>
+    <!-- <xacro:VLP-16R parent="base_footprint" name="velodyne" topic="/velodyne_points" hz="10" samples="800" active="$(arg simulate_perception)"> -->
+	<!-- <origin xyz="0.59 0.0 0.30" rpy="0 0 0"/> -->
+    <!-- </xacro:VLP-16R> -->
+    <xacro:VLP-16 parent="base_footprint" name="velodyne" topic="/velodyne_points" organize_cloud="false" hz="10" samples="440" gpu="false">
+        <origin xyz="0.59 0.0 0.30" rpy="0 0 0" />
+    </xacro:VLP-16>
     <xacro:zed_camera parent="base_footprint" prefix="zed" active="$(arg simulate_perception)">
 	<origin xyz="0.12 0.0 0.76" rpy="0 ${10.15*M_PI/180.0} 0"/>

File: eufs_racecar/robots/eufs/robot.urdf.xacro (robot description, xacro)
@@ -46,7 +46,10 @@
         <origin xyz="0.0 0.0 0.4" rpy="0 0 0"/>
     </xacro:sensor_gps>
-    <xacro:VLP-16R parent="base_footprint" name="velodyne" topic="/velodyne_points" hz="10" active="$(arg simulate_perception)">
-        <origin xyz="-0.15 0.0 0.30" rpy="0 0 0"/>
-    </xacro:VLP-16R>
+    <!-- <xacro:VLP-16R parent="base_footprint" name="velodyne" topic="/velodyne_points" hz="10" active="$(arg simulate_perception)"> -->
+        <!-- <origin xyz="-0.15 0.0 0.30" rpy="0 0 0"/> -->
+    <!-- </xacro:VLP-16R> -->
+    <xacro:VLP-16 parent="base_footprint" name="velodyne" topic="/velodyne_points" organize_cloud="false" hz="10" samples="440" gpu="false">
+        <origin xyz="-0.15 0.0 0.30" rpy="0 0 0" />
+    </xacro:VLP-16>
     <xacro:zed_camera parent="base_footprint" prefix="zed" active="$(arg simulate_perception)">
         <origin xyz="-0.08 0.0 0.76" rpy="0 0 0"/>

File: eufs_sensors/urdf/all_sensors.urdf.xacro (robot description, xacro)
@@ -5,5 +5,6 @@
   <xacro:include filename="$(find eufs_sensors)/urdf/gps.urdf.xacro"/>
   <!-- Velodyne VLP-16R -->
-  <xacro:include filename="$(find eufs_sensors)/urdf/VLP-16R.urdf.xacro"/>
+  <!-- <xacro:include filename="$(find eufs_sensors)/urdf/VLP-16R.urdf.xacro"/> -->
+  <xacro:include filename="$(find velodyne_description)/urdf/VLP-16.urdf.xacro"/>
   <!-- Imu -->
   <xacro:include filename="$(find eufs_sensors)/urdf/imu.urdf.xacro"/>
